File: pcb/pcb.sch (KiCad schematic (older format))
At the start: 10 parts

Commit message: Adds type-c ai03 library, continues work on schematic
Parts:
- added C? (x2): 22pF, symbol Device:C_Small
- added F?: 500mA, symbol Device:Polyfuse
- added R?: 10k, symbol Device:R_Small
- added SW?: SW_PUSH, symbol kbd:SW_PUSH
- added USB?: HRO-TYPE-C-31-M-12, symbol Type-C:HRO-TYPE-C-31-M-12
- Y?: value Crystal_GND24_Small -> 16MHz
Connections:
- net labels added: D+, D-, VCC
- wire segments 24 -> 49
Changed lines of the file:
@@
 P 1550 4000
 F 0 "Y?" V 1504 4144 50  0000 L CNN
-F 1 "Crystal_GND24_Small" V 1595 4144 50  0000 L CNN
+F 1 "16MHz" V 1595 4144 50  0000 L CNN
 F 2 "" H 1550 4000 50  0001 C CNN
 F 3 "~" H 1550 4000 50  0001 C CNN
@@
 Wire Wire Line
 	2200 4100 1550 4100
+$Comp
+L Device:C_Small C?
+U 1 1 5F3B53EA
+P 1250 3800
+F 0 "C?" V 1021 3800 50  0000 C CNN
+F 1 "22pF" V 1112 3800 50  0000 C CNN
+F 2 "" H 1250 3800 50  0001 C CNN
+F 3 "~" H 1250 3800 50  0001 C CNN
+	1    1250 3800
+	0    1    1    0
+$EndComp
+$Comp
+L Device:C_Small C?
+U 1 1 5F3B7682
+P 1250 4200
+F 0 "C?" V 1021 4200 50  0000 C CNN
+F 1 "22pF" V 1112 4200 50  0000 C CNN
+F 2 "" H 1250 4200 50  0001 C CNN
+F 3 "~" H 1250 4200 50  0001 C CNN
+	1    1250 4200
+	0    1    1    0
+$EndComp
+$Comp
+L power:GND #PWR?
+U 1 1 5F3B840D
+P 1150 4350
+F 0 "#PWR?" H 1150 4100 50  0001 C CNN
+F 1 "GND" H 1155 4177 50  0000 C CNN
+F 2 "" H 1150 4350 50  0001 C CNN
+F 3 "" H 1150 4350 50  0001 C CNN
+	1    1150 4350
+	1    0    0    -1
+$EndComp
+Wire Wire Line
+	1150 4350 1150 4200
+Connection ~ 1150 4200
+Wire Wire Line
+	1150 4200 1150 3800
+Wire Wire Line
+	1350 3800 1550 3800
+Wire Wire Line
+	1550 3800 1550 3900
+Connection ~ 1550 3900
+Wire Wire Line
+	1450 4000 1450 4250
+Wire Wire Line
+	1450 4350 1150 4350
+Connection ~ 1150 4350
+Wire Wire Line
+	1550 4100 1550 4250
+Wire Wire Line
+	1550 4250 1450 4250
+Connection ~ 1550 4100
+Connection ~ 1450 4250
+Wire Wire Line
+	1450 4250 1450 4350
+Wire Wire Line
+	1350 4200 1350 4100
+Wire Wire Line
+	1350 4100 1550 4100
+$Comp
+L kbd:SW_PUSH SW?
+U 1 1 5F3BD178
+P 1800 3700
+F 0 "SW?" H 1800 3955 50  0000 C CNN
+F 1 "SW_PUSH" H 1800 3864 50  0000 C CNN
+F 2 "" H 1800 3700 50  0000 C CNN
+F 3 "" H 1800 3700 50  0000 C CNN
+	1    1800 3700
+	1    0    0    -1
+$EndComp
+$Comp
+L power:GND #PWR?
+U 1 1 5F3BD7AF
+P 1400 3400
+F 0 "#PWR?" H 1400 3150 50  0001 C CNN
+F 1 "GND" H 1405 3227 50  0000 C CNN
+F 2 "" H 1400 3400 50  0001 C CNN
+F 3 "" H 1400 3400 50  0001 C CNN
+	1    1400 3400
+	1    0    0    -1
+$EndComp
+Wire Wire Line
+	1400 3400 1500 3400
+Wire Wire Line
+	1500 3400 1500 3700
+Wire Wire Line
+	2100 3700 2150 3700
+$Comp
+L Device:R_Small R?
+U 1 1 5F3BF8EA
+P 2150 3200
+F 0 "R?" H 2209 3246 50  0000 L CNN
+F 1 "10k" H 2209 3155 50  0000 L CNN
+F 2 "" H 2150 3200 50  0001 C CNN
+F 3 "~" H 2150 3200 50  0001 C CNN
+	1    2150 3200
+	1    0    0    -1
+$EndComp
+$Comp
+L power:+5V #PWR?
+U 1 1 5F3BFF46
+P 2150 3000
+F 0 "#PWR?" H 2150 2850 50  0001 C CNN
+F 1 "+5V" H 2165 3173 50  0000 C CNN
+F 2 "" H 2150 3000 50  0001 C CNN
+F 3 "" H 2150 3000 50  0001 C CNN
+	1    2150 3000
+	1    0    0    -1
+$EndComp
+Wire Wire Line
+	2150 3000 2150 3100
+Wire Wire Line
+	2150 3300 2150 3700
+Connection ~ 2150 3700
+Wire Wire Line
+	2150 3700 2200 3700
+Text GLabel 750  4700 0    50   Input ~ 0
+D+
+Text GLabel 750  4800 0    50   Input ~ 0
+D-
+$Comp
+L Type-C:HRO-TYPE-C-31-M-12 USB?
+U 1 1 5F3C8A31
+P 1450 1600
+F 0 "USB?" H 1283 2397 60  0000 C CNN
+F 1 "HRO-TYPE-C-31-M-12" H 1283 2291 60  0000 C CNN
+F 2 "" H 1450 1600 60  0001 C CNN
+F 3 "" H 1450 1600 60  0001 C CNN
+	1    1450 1600
+	1    0    0    -1
+$EndComp
+$Comp
+L power:GND #PWR?
+U 1 1 5F3CA697
+P 1900 2250
+F 0 "#PWR?" H 1900 2000 50  0001 C CNN
+F 1 "GND" H 1905 2077 50  0000 C CNN
+F 2 "" H 1900 2250 50  0001 C CNN
+F 3 "" H 1900 2250 50  0001 C CNN
+	1    1900 2250
+	1    0    0    -1
+$EndComp
+Wire Wire Line
+	1550 2250 1900 2250
+Wire Wire Line
+	1550 2150 1900 2150
+Wire Wire Line
+	1900 2150 1900 2250
+Connection ~ 1900 2250
+$Comp
+L power:VCC #PWR?
+U 1 1 5F3CCB5D
+P 2250 1150
+F 0 "#PWR?" H 2250 1000 50  0001 C CNN
+F 1 "VCC" H 2267 1323 50  0000 C CNN
+F 2 "" H 2250 1150 50  0001 C CNN
+F 3 "" H 2250 1150 50  0001 C CNN
+	1    2250 1150
+	1    0    0    -1
+$EndComp
+Wire Wire Line
+	1550 1050 1900 1050
+Wire Wire Line
+	1900 1050 1900 2150
+Connection ~ 1900 2150
+Wire Wire Line
+	1550 1150 2250 1150
+$Comp
+L Device:Polyfuse F?
+U 1 1 5F3D0F13
+P 2600 1150
+F 0 "F?" V 2375 1150 50  0000 C CNN
+F 1 "500mA" V 2466 1150 50  0000 C CNN
+F 2 "" H 2650 950 50  0001 L CNN
+F 3 "~" H 2600 1150 50  0001 C CNN
+	1    2600 1150
+	0    1    1    0
+$EndComp
+$Comp
+L power:+5V #PWR?
+U 1 1 5F3D1EE1
+P 3150 1150
+F 0 "#PWR?" H 3150 1000 50  0001 C CNN
+F 1 "+5V" H 3165 1323 50  0000 C CNN
+F 2 "" H 3150 1150 50  0001 C CNN
+F 3 "" H 3150 1150 50  0001 C CNN
+	1    3150 1150
+	1    0    0    -1
+$EndComp
+Wire Wire Line
+	3150 1150 2750 1150
+Wire Wire Line
+	2450 1150 2250 1150
+Connection ~ 2250 1150
 $EndSCHEMATC

Commit message: Completes schematic, adds more submodules
Parts:
- added D1, D10, D11, D12, D13, D14, D15, D16, D17, D18, D19, D2, D20, D21, D22, D23, D24, D25, D26, D27, D28, D29, D3, D30, D31, D32, D4, D5, D6, D7, D8, D9: SOD_123, Diode_SMD:D_SOD-123, symbol Device:D_Small
- added OL1: OLED, kbd:OLED_1side, symbol kbd:OLED
- added R2, R3: 10k, Resistor_SMD:R_0805_2012Metric, symbol Device:R_Small
- added R7, R8: 5k1, Resistor_SMD:R_0805_2012Metric, symbol Device:R_Small
- added SW1, SW10, SW11, SW12, SW13, SW14, SW15, SW16, SW17, SW18, SW19, SW2, SW20, SW21, SW22, SW23, SW24, SW25, SW26, SW27, SW28, SW29, SW3, SW30, SW31, SW32, SW4, SW5, SW6, SW7, SW8, SW9: SW_PUSH, kbd:CherryMX_Choc_Hotswap, symbol kbd:SW_PUSH
- added SW33: Rotary_Encoder, Keebio-Parts:RotaryEncoder_EC11, symbol Device:Rotary_Encoder
- C1, C2, C3, C4, C5, C6, C7: renamed from C?; footprint (none) -> Capacitor_SMD:C_0805_2012Metric
- F1: renamed from F?; footprint (none) -> Fuse:Fuse_1206_3216Metric
- R1, R4, R5, R6: renamed from R?; footprint (none) -> Resistor_SMD:R_0805_2012Metric
- SW34: renamed from SW?; footprint (none) -> Button_Switch_SMD:SW_SPST_B3U-1000P
- USB1: renamed from USB?; footprint (none) -> Type-C:HRO-TYPE-C-31-M-12-HandSoldering
- Y1: renamed from Y?; footprint (none) -> Crystal:Crystal_SMD_3225-4Pin_3.2x2.5mm
- gave numbers to parts that had none: 1
Connections:
- net labels added: COL0, COL1, COL2, COL3, COL4, COL5, COL6, COL7, COL8, COL9, ROW0, ROW1, ROW2, ROW3, S0, S1, SCL, SDA
- wire segments 49 -> 178

Commit message: Moves some submodules around, completes placement of components.
Parts:
- SW1, SW10, SW11, SW12, SW13, SW14, SW15, SW16, SW17, SW18, SW19, SW2, SW20, SW21, SW22, SW23, SW24, SW25, SW26, SW27, SW28, SW29, SW3, SW30, SW4, SW5, SW6, SW7, SW8, SW9: footprint kbd:CherryMX_Choc_Hotswap -> MX_Only:MXOnly-1U
- SW31, SW32: footprint kbd:CherryMX_Choc_Hotswap -> MX_Only:MXOnly-2U
Changed lines of the file:
@@
 F 0 "SW1" H 3850 2205 50  0000 C CNN
 F 1 "SW_PUSH" H 3850 2114 50  0000 C CNN
-F 2 "kbd:CherryMX_Choc_Hotswap" H 3850 1950 50  0001 C CNN
+F 2 "MX_Only:MXOnly-1U" H 3850 1950 50  0001 C CNN
 F 3 "" H 3850 1950 50  0000 C CNN
 	1    3850 1950
@@
 F 0 "SW11" H 3850 2655 50  0000 C CNN
 F 1 "SW_PUSH" H 3850 2564 50  0000 C CNN
-F 2 "kbd:CherryMX_Choc_Hotswap" H 3850 2400 50  0001 C CNN
+F 2 "MX_Only:MXOnly-1U" H 3850 2400 50  0001 C CNN
 F 3 "" H 3850 2400 50  0000 C CNN
 	1    3850 2400
@@
 F 0 "SW21" H 3850 3105 50  0000 C CNN
 F 1 "SW_PUSH" H 3850 3014 50  0000 C CNN
-F 2 "kbd:CherryMX_Choc_Hotswap" H 3850 2850 50  0001 C CNN
+F 2 "MX_Only:MXOnly-1U" H 3850 2850 50  0001 C CNN
 F 3 "" H 3850 2850 50  0000 C CNN
 	1    3850 2850
@@
 F 0 "SW2" H 4550 2205 50  0000 C CNN
 F 1 "SW_PUSH" H 4550 2114 50  0000 C CNN
-F 2 "kbd:CherryMX_Choc_Hotswap" H 4550 1950 50  0001 C CNN
+F 2 "MX_Only:MXOnly-1U" H 4550 1950 50  0001 C CNN
 F 3 "" H 4550 1950 50  0000 C CNN
 	1    4550 1950
@@
 F 0 "SW3" H 5250 2205 50  0000 C CNN
 F 1 "SW_PUSH" H 5250 2114 50  0000 C CNN
-F 2 "kbd:CherryMX_Choc_Hotswap" H 5250 1950 50  0001 C CNN
+F 2 "MX_Only:MXOnly-1U" H 5250 1950 50  0001 C CNN
 F 3 "" H 5250 1950 50  0000 C CNN
 	1    5250 1950
@@
 F 0 "SW4" H 5950 2205 50  0000 C CNN
 F 1 "SW_PUSH" H 5950 2114 50  0000 C CNN
-F 2 "kbd:CherryMX_Choc_Hotswap" H 5950 1950 50  0001 C CNN
+F 2 "MX_Only:MXOnly-1U" H 5950 1950 50  0001 C CNN
 F 3 "" H 5950 1950 50  0000 C CNN
 	1    5950 1950
@@
 F 0 "SW5" H 6650 2205 50  0000 C CNN
 F 1 "SW_PUSH" H 6650 2114 50  0000 C CNN
-F 2 "kbd:CherryMX_Choc_Hotswap" H 6650 1950 50  0001 C CNN
+F 2 "MX_Only:MXOnly-1U" H 6650 1950 50  0001 C CNN
 F 3 "" H 6650 1950 50  0000 C CNN
 	1    6650 1950
@@
 F 0 "SW12" H 4550 2655 50  0000 C CNN
 F 1 "SW_PUSH" H 4550 2564 50  0000 C CNN
-F 2 "kbd:CherryMX_Choc_Hotswap" H 4550 2400 50  0001 C CNN
+F 2 "MX_Only:MXOnly-1U" H 4550 2400 50  0001 C CNN
 F 3 "" H 4550 2400 50  0000 C CNN
 	1    4550 2400
@@
 F 0 "SW13" H 5250 2655 50  0000 C CNN
 F 1 "SW_PUSH" H 5250 2564 50  0000 C CNN
-F 2 "kbd:CherryMX_Choc_Hotswap" H 5250 2400 50  0001 C CNN
+F 2 "MX_Only:MXOnly-1U" H 5250 2400 50  0001 C CNN
 F 3 "" H 5250 2400 50  0000 C CNN
 	1    5250 2400
@@
 F 0 "SW14" H 5950 2655 50  0000 C CNN
 F 1 "SW_PUSH" H 5950 2564 50  0000 C CNN
-F 2 "kbd:CherryMX_Choc_Hotswap" H 5950 2400 50  0001 C CNN
+F 2 "MX_Only:MXOnly-1U" H 5950 2400 50  0001 C CNN
 F 3 "" H 5950 2400 50  0000 C CNN
 	1    5950 2400
@@
 F 0 "SW15" H 6650 2655 50  0000 C CNN
 F 1 "SW_PUSH" H 6650 2564 50  0000 C CNN
-F 2 "kbd:CherryMX_Choc_Hotswap" H 6650 2400 50  0001 C CNN
+F 2 "MX_Only:MXOnly-1U" H 6650 2400 50  0001 C CNN
 F 3 "" H 6650 2400 50  0000 C CNN
 	1    6650 2400
@@
 F 0 "SW22" H 4550 3105 50  0000 C CNN
 F 1 "SW_PUSH" H 4550 3014 50  0000 C CNN
-F 2 "kbd:CherryMX_Choc_Hotswap" H 4550 2850 50  0001 C CNN
+F 2 "MX_Only:MXOnly-1U" H 4550 2850 50  0001 C CNN
 F 3 "" H 4550 2850 50  0000 C CNN
 	1    4550 2850
@@
 F 0 "SW23" H 5250 3105 50  0000 C CNN
 F 1 "SW_PUSH" H 5250 3014 50  0000 C CNN
-F 2 "kbd:CherryMX_Choc_Hotswap" H 5250 2850 50  0001 C CNN
+F 2 "MX_Only:MXOnly-1U" H 5250 2850 50  0001 C CNN
 F 3 "" H 5250 2850 50  0000 C CNN
 	1    5250 2850
@@
 F 0 "SW24" H 5950 3105 50  0000 C CNN
 F 1 "SW_PUSH" H 5950 3014 50  0000 C CNN
-F 2 "kbd:CherryMX_Choc_Hotswap" H 5950 2850 50  0001 C CNN
+F 2 "MX_Only:MXOnly-1U" H 5950 2850 50  0001 C CNN
 F 3 "" H 5950 2850 50  0000 C CNN
 	1    5950 2850
@@
 F 0 "SW25" H 6650 3105 50  0000 C CNN
 F 1 "SW_PUSH" H 6650 3014 50  0000 C CNN
-F 2 "kbd:CherryMX_Choc_Hotswap" H 6650 2850 50  0001 C CNN
+F 2 "MX_Only:MXOnly-1U" H 6650 2850 50  0001 C CNN
 F 3 "" H 6650 2850 50  0000 C CNN
 	1    6650 2850
@@
 F 0 "SW31" H 6650 3505 50  0000 C CNN
 F 1 "SW_PUSH" H 6650 3414 50  0000 C CNN
-F 2 "kbd:CherryMX_Choc_Hotswap" H 6650 3250 50  0001 C CNN
+F 2 "MX_Only:MXOnly-2U" H 6650 3250 50  0001 C CNN
 F 3 "" H 6650 3250 50  0000 C CNN
 	1    6650 3250
@@
 F 0 "SW32" H 7500 3505 50  0000 C CNN
 F 1 "SW_PUSH" H 7500 3414 50  0000 C CNN
-F 2 "kbd:CherryMX_Choc_Hotswap" H 7500 3250 50  0001 C CNN
+F 2 "MX_Only:MXOnly-2U" H 7500 3250 50  0001 C CNN
 F 3 "" H 7500 3250 50  0000 C CNN
 	1    7500 3250
@@
 F 0 "SW26" H 7500 3105 50  0000 C CNN
 F 1 "SW_PUSH" H 7500 3014 50  0000 C CNN
-F 2 "kbd:CherryMX_Choc_Hotswap" H 7500 2850 50  0001 C CNN
+F 2 "MX_Only:MXOnly-1U" H 7500 2850 50  0001 C CNN
 F 3 "" H 7500 2850 50  0000 C CNN
 	1    7500 2850
@@
 F 0 "SW16" H 7500 2655 50  0000 C CNN
 F 1 "SW_PUSH" H 7500 2564 50  0000 C CNN
-F 2 "kbd:CherryMX_Choc_Hotswap" H 7500 2400 50  0001 C CNN
+F 2 "MX_Only:MXOnly-1U" H 7500 2400 50  0001 C CNN
 F 3 "" H 7500 2400 50  0000 C CNN
 	1    7500 2400
@@
 F 0 "SW6" H 7500 2205 50  0000 C CNN
 F 1 "SW_PUSH" H 7500 2114 50  0000 C CNN
-F 2 "kbd:CherryMX_Choc_Hotswap" H 7500 1950 50  0001 C CNN
+F 2 "MX_Only:MXOnly-1U" H 7500 1950 50  0001 C CNN
 F 3 "" H 7500 1950 50  0000 C CNN
 	1    7500 1950
@@
 F 0 "SW7" H 8250 2205 50  0000 C CNN
 F 1 "SW_PUSH" H 8250 2114 50  0000 C CNN
-F 2 "kbd:CherryMX_Choc_Hotswap" H 8250 1950 50  0001 C CNN
+F 2 "MX_Only:MXOnly-1U" H 8250 1950 50  0001 C CNN
 F 3 "" H 8250 1950 50  0000 C CNN
 	1    8250 1950
@@
 F 0 "SW17" H 8250 2655 50  0000 C CNN
 F 1 "SW_PUSH" H 8250 2564 50  0000 C CNN
-F 2 "kbd:CherryMX_Choc_Hotswap" H 8250 2400 50  0001 C CNN
+F 2 "MX_Only:MXOnly-1U" H 8250 2400 50  0001 C CNN
 F 3 "" H 8250 2400 50  0000 C CNN
 	1    8250 2400
@@
 F 0 "SW27" H 8250 3105 50  0000 C CNN
 F 1 "SW_PUSH" H 8250 3014 50  0000 C CNN
-F 2 "kbd:CherryMX_Choc_Hotswap" H 8250 2850 50  0001 C CNN
+F 2 "MX_Only:MXOnly-1U" H 8250 2850 50  0001 C CNN
 F 3 "" H 8250 2850 50  0000 C CNN
 	1    8250 2850
@@
 F 0 "SW28" H 9000 3105 50  0000 C CNN
 F 1 "SW_PUSH" H 9000 3014 50  0000 C CNN
-F 2 "kbd:CherryMX_Choc_Hotswap" H 9000 2850 50  0001 C CNN
+F 2 "MX_Only:MXOnly-1U" H 9000 2850 50  0001 C CNN
 F 3 "" H 9000 2850 50  0000 C CNN
 	1    9000 2850
@@
 F 0 "SW18" H 9000 2655 50  0000 C CNN
 F 1 "SW_PUSH" H 9000 2564 50  0000 C CNN
-F 2 "kbd:CherryMX_Choc_Hotswap" H 9000 2400 50  0001 C CNN
+F 2 "MX_Only:MXOnly-1U" H 9000 2400 50  0001 C CNN
 F 3 "" H 9000 2400 50  0000 C CNN
 	1    9000 2400
@@
 F 0 "SW8" H 9000 2205 50  0000 C CNN
 F 1 "SW_PUSH" H 9000 2114 50  0000 C CNN
-F 2 "kbd:CherryMX_Choc_Hotswap" H 9000 1950 50  0001 C CNN
+F 2 "MX_Only:MXOnly-1U" H 9000 1950 50  0001 C CNN
 F 3 "" H 9000 1950 50  0000 C CNN
 	1    9000 1950
@@
 F 0 "SW9" H 9700 2205 50  0000 C CNN
 F 1 "SW_PUSH" H 9700 2114 50  0000 C CNN
-F 2 "kbd:CherryMX_Choc_Hotswap" H 9700 1950 50  0001 C CNN
+F 2 "MX_Only:MXOnly-1U" H 9700 1950 50  0001 C CNN
 F 3 "" H 9700 1950 50  0000 C CNN
 	1    9700 1950
@@
 F 0 "SW10" H 10400 2205 50  0000 C CNN
 F 1 "SW_PUSH" H 10400 2114 50  0000 C CNN
-F 2 "kbd:CherryMX_Choc_Hotswap" H 10400 1950 50  0001 C CNN
+F 2 "MX_Only:MXOnly-1U" H 10400 1950 50  0001 C CNN
 F 3 "" H 10400 1950 50  0000 C CNN
 	1    10400 1950
@@
 F 0 "SW19" H 9700 2655 50  0000 C CNN
 F 1 "SW_PUSH" H 9700 2564 50  0000 C CNN
-F 2 "kbd:CherryMX_Choc_Hotswap" H 9700 2400 50  0001 C CNN
+F 2 "MX_Only:MXOnly-1U" H 9700 2400 50  0001 C CNN
 F 3 "" H 9700 2400 50  0000 C CNN
 	1    9700 2400
@@
 F 0 "SW20" H 10400 2655 50  0000 C CNN
 F 1 "SW_PUSH" H 10400 2564 50  0000 C CNN
-F 2 "kbd:CherryMX_Choc_Hotswap" H 10400 2400 50  0001 C CNN
+F 2 "MX_Only:MXOnly-1U" H 10400 2400 50  0001 C CNN
 F 3 "" H 10400 2400 50  0000 C CNN
 	1    10400 2400
@@
 F 0 "SW30" H 10400 3105 50  0000 C CNN
 F 1 "SW_PUSH" H 10400 3014 50  0000 C CNN
-F 2 "kbd:CherryMX_Choc_Hotswap" H 10400 2850 50  0001 C CNN
+F 2 "MX_Only:MXOnly-1U" H 10400 2850 50  0001 C CNN
 F 3 "" H 10400 2850 50  0000 C CNN
 	1    10400 2850
@@
 F 0 "SW29" H 9700 3105 50  0000 C CNN
 F 1 "SW_PUSH" H 9700 3014 50  0000 C CNN
-F 2 "kbd:CherryMX_Choc_Hotswap" H 9700 2850 50  0001 C CNN
+F 2 "MX_Only:MXOnly-1U" H 9700 2850 50  0001 C CNN
 F 3 "" H 9700 2850 50  0000 C CNN
 	1    9700 2850

Commit message: Continues working on routing, moved to using some different components
Parts:
- removed C1: 10uF, Capacitor_SMD:C_0805_2012Metric, symbol Device:C_Small
- removed C2, C3, C4: 0.1uF, Capacitor_SMD:C_0805_2012Metric, symbol Device:C_Small
- removed C5: 1uF, Capacitor_SMD:C_0805_2012Metric, symbol Device:C_Small
- removed C6, C7: 22pF, Capacitor_SMD:C_0805_2012Metric, symbol Device:C_Small
- removed F1: 500mA, Fuse:Fuse_1206_3216Metric, symbol Device:Polyfuse
- removed R1, R2, R3, R4: 10k, Resistor_SMD:R_0805_2012Metric, symbol Device:R_Small
- removed R5, R6: 22, Resistor_SMD:R_0805_2012Metric, symbol Device:R_Small
- removed R7, R8: 5k1, Resistor_SMD:R_0805_2012Metric, symbol Device:R_Small
- removed U1: ATmega32U4-AU, Package_QFP:TQFP-44_10x10mm_P0.8mm, symbol MCU_Microchip_ATmega:ATmega32U4-AU
- removed USB1: HRO-TYPE-C-31-M-12, Type-C:HRO-TYPE-C-31-M-12-HandSoldering, symbol Type-C:HRO-TYPE-C-31-M-12
- removed Y1: 16MHz, Crystal:Crystal_SMD_3225-4Pin_3.2x2.5mm, symbol Device:Crystal_GND24_Small
- added U1: ProMicro, kbd:ProMicro_v3.5, symbol kbd:ProMicro
- D1, D10, D11, D12, D13, D14, D15, D16, D17, D18, D19, D2, D20, D21, D22, D23, D24, D25, D26, D27, D28, D29, D3, D30, D31, D32, D4, D5, D6, D7, D8, D9: footprint Diode_SMD:D_SOD-123 -> kbd:D3_TH
- SW1, SW10, SW11, SW12, SW13, SW14, SW15, SW16, SW17, SW18, SW19, SW2, SW20, SW21, SW22, SW23, SW24, SW25, SW26, SW27, SW28, SW29, SW3, SW30, SW4, SW5, SW6, SW7, SW8, SW9: footprint MX_Only:MXOnly-1U -> MX_Only:MXOnly-1U-NoLED
- SW31, SW32: footprint MX_Only:MXOnly-2U -> MX_Only:MXOnly-2U-NoLED
- SW34: footprint Button_Switch_SMD:SW_SPST_B3U-1000P -> kbd:ResetSW_1side
Connections:
- net labels added: reset
- net labels removed: +5V, D+, D-
- wire segments 178 -> 110
Other:
- moved on the sheet: D1, D10, D11, D12, D13, D14, D15, D16, D17, D18, D19, D2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

Commit message: Finishes routing
Connections:
- net COL0: now also SW16.1, SW26.1, SW32.1, SW6.1, U1.20 (F4/A3); no longer U1.11 (8/B4)
- net COL1: now also SW17.1, SW27.1, SW7.1, U1.19 (F5/A2); no longer U1.12 (9/B5)
- net COL2: now also SW18.1, SW28.1, SW8.1, U1.18 (F6/A1); no longer U1.20 (F4/A3)
- net COL3: now also SW19.1, SW29.1, SW9.1, U1.17 (F7/A0); no longer U1.19 (F5/A2)
- net COL4: now also SW10.1, SW20.1, SW30.1, U1.16 (B1/15); no longer U1.18 (F6/A1)
- net S0: now also U1.11 (8/B4); no longer U1.1 (TX0/D3)
- net S1: now also U1.12 (9/B5); no longer U1.2 (RX1/D2)
- removed net COL5: SW16.1, SW26.1, SW32.1, SW6.1, U1.17 (F7/A0)
- removed net COL6: SW17.1, SW27.1, SW7.1, U1.16 (B1/15)
- removed net COL7: SW18.1, SW28.1, SW8.1, U1.15 (B3/14)
- removed net COL8: SW19.1, SW29.1, SW9.1, U1.14 (B2/16)
- removed net COL9: SW10.1, SW20.1, SW30.1, U1.13 (B6/10)
Changed lines of the file:
@@
 COL4
 Text GLabel 6000 1000 1    50   Input ~ 0
-COL5
+COL0
 Text GLabel 6750 1000 1    50   Input ~ 0
-COL6
+COL1
 Text GLabel 7500 1000 1    50   Input ~ 0
-COL7
+COL2
 Text GLabel 8200 1000 1    50   Input ~ 0
-COL8
+COL3
 Text GLabel 8900 1000 1    50   Input ~ 0
-COL9
+COL4
 Text GLabel 1950 1700 3    50   Input ~ 0
 ROW0
@@
 	1    0    0    -1
 $EndComp
-Text GLabel 1750 4800 0    50   Input ~ 0
+Text GLabel 1750 5800 0    50   Input ~ 0
 S0
 Wire Wire Line
@@
 Text GLabel 2200 4150 0    50   Input ~ 0
 reset
-Text GLabel 1750 4900 0    50   Input ~ 0
+Text GLabel 1750 5900 0    50   Input ~ 0
 S1
+Text GLabel 3150 5600 2    50   Input ~ 0
+COL4
 Text GLabel 3150 5500 2    50   Input ~ 0
-COL5
-Text GLabel 3150 5600 2    50   Input ~ 0
-COL6
-Text GLabel 3150 5700 2    50   Input ~ 0
-COL7
+COL3
 Text GLabel 3150 5400 2    50   Input ~ 0
-COL4
+COL2
 Text GLabel 3150 5300 2    50   Input ~ 0
-COL3
+COL1
 Text GLabel 3150 5200 2    50   Input ~ 0
-COL2
-Text GLabel 1750 5900 0    50   Input ~ 0
-COL1
-Text GLabel 1750 5800 0    50   Input ~ 0
 COL0
 Text GLabel 1750 5700 0    50   Input ~ 0
@@
 Text GLabel 1750 5200 0    50   Input ~ 0
 SDA
-Text GLabel 3150 5800 2    50   Input ~ 0
-COL8
-Text GLabel 3150 5900 2    50   Input ~ 0
-COL9
 Wire Wire Line
 	6600 2950 5750 2950
