File: pcb/pcb.sch (KiCad schematic (older format))
At the start: 70 parts, among them SW1 SW_PUSH, SW10 SW_PUSH, SW11 SW_PUSH, SW12 SW_PUSH, SW13 SW_PUSH, SW14 SW_PUSH, SW15 SW_PUSH, SW16 SW_PUSH, SW17 SW_PUSH, SW18 SW_PUSH, SW19 SW_PUSH, SW2 SW_PUSH, SW20 SW_PUSH, SW21 SW_PUSH, SW22 SW_PUSH, SW23 SW_PUSH, SW24 SW_PUSH, SW25 SW_PUSH, SW26 SW_PUSH, SW27 SW_PUSH, SW28 SW_PUSH, SW29 SW_PUSH, SW3 SW_PUSH, SW30 SW_PUSH, SW31 SW_PUSH, SW32 SW_PUSH, SW33 Rotary_Encoder_Switch, SW34 SW_PUSH, SW4 SW_PUSH, SW5 SW_PUSH, SW6 SW_PUSH, SW7 SW_PUSH, SW8 SW_PUSH, SW9 SW_PUSH, U1 ProMicro

Commit message: Finishes move back to pro micro, adds silk footprint and lib, updates routing, fixes outline
Parts:
- D1, D10, D11, D12, D13, D14, D15, D16, D17, D18, D19, D2, D20, D21, D22, D23, D24, D25, D26, D27, D28, D29, D3, D30, D31, D32, D4, D5, D6, D7, D8, D9: symbol Device:D_Small -> pcb-rescue:D_Small-Device
- OL1: symbol kbd:OLED -> pcb-rescue:OLED-kbd
- R1, R2: symbol Device:R_Small -> pcb-rescue:R_Small-Device
- SW1, SW10, SW11, SW12, SW13, SW14, SW15, SW16, SW17, SW18, SW19, SW2, SW20, SW21, SW22, SW23, SW24, SW25, SW26, SW27, SW28, SW29, SW3, SW30, SW31, SW32, SW34, SW4, SW5, SW6, SW7, SW8, SW9: symbol kbd:SW_PUSH -> pcb-rescue:SW_PUSH-kbd
- SW33: symbol Device:Rotary_Encoder_Switch -> pcb-rescue:Rotary_Encoder_Switch-Device
- U1: symbol kbd:ProMicro -> pcb-rescue:ProMicro-kbd
