File: pcb/pcb.sch (KiCad schematic (older format))
At the start: 70 parts, among them SW1 SW_PUSH, SW10 SW_PUSH, SW11 SW_PUSH, SW12 SW_PUSH, SW13 SW_PUSH, SW14 SW_PUSH, SW15 SW_PUSH, SW16 SW_PUSH, SW17 SW_PUSH, SW18 SW_PUSH, SW19 SW_PUSH, SW2 SW_PUSH, SW20 SW_PUSH, SW21 SW_PUSH, SW22 SW_PUSH, SW23 SW_PUSH, SW24 SW_PUSH, SW25 SW_PUSH, SW26 SW_PUSH, SW27 SW_PUSH, SW28 SW_PUSH, SW29 SW_PUSH, SW3 SW_PUSH, SW30 SW_PUSH, SW31 SW_PUSH, SW32 SW_PUSH, SW33 Rotary_Encoder_Switch, SW34 SW_PUSH, SW4 SW_PUSH, SW5 SW_PUSH, SW6 SW_PUSH, SW7 SW_PUSH, SW8 SW_PUSH, SW9 SW_PUSH, U1 ProMicro

Commit message: Updates kawa to remove encoder, adds new oled footprint, reroute accordingly
Parts:
- removed OL1: OLED, kbd:OLED_1side, symbol pcb-rescue:OLED-kbd
- removed SW33: Rotary_Encoder_Switch, keebio-parts:RotaryEncoder_EC11, symbol pcb-rescue:Rotary_Encoder_Switch-Device
- added Brd1: SSD1306, SSD1306:128x64OLED, symbol SSD1306-128x64_OLED:SSD1306
Connections:
- net labels removed: S0, S1
- wire segments 123 -> 116
- no-connect marks 0 -> 3
Changed lines of the file:
@@
 Comment4 ""
 $EndDescr
-$Comp
-L pcb-rescue:OLED-kbd OL1
-U 1 1 5F3A39E2
-P 3300 3300
-F 0 "OL1" H 3928 3369 51  0000 L CNN
-F 1 "OLED" H 3928 3279 47  0000 L CNN
-F 2 "kbd:OLED_1side" H 3300 3400 60  0001 C CNN
-F 3 "" H 3300 3400 60  0001 C CNN
-	1    3300 3300
-	1    0    0    -1
-$EndComp
-$Comp
-L pcb-rescue:GND-power #PWR0115
-U 1 1 5F4567A6
-P 1750 3500
-F 0 "#PWR0115" H 1750 3250 50  0001 C CNN
-F 1 "GND" H 1755 3327 50  0000 C CNN
-F 2 "" H 1750 3500 50  0001 C CNN
-F 3 "" H 1750 3500 50  0001 C CNN
-	1    1750 3500
-	1    0    0    -1
-$EndComp
-Wire Wire Line
-	1750 3500 2550 3500
-Wire Wire Line
-	2550 3350 1750 3350
-Text GLabel 2150 3200 0    50   Input ~ 0
-SCL
-Wire Wire Line
-	2550 3200 2150 3200
-Text GLabel 2150 3050 0    50   Input ~ 0
+Wire Wire Line
+	2650 3300 1850 3300
+Text GLabel 2250 3100 0    50   Input ~ 0
 SDA
-Wire Wire Line
-	2150 3050 2550 3050
 $Comp
 L pcb-rescue:SW_PUSH-kbd SW1
@@
 $EndComp
 $Comp
-L pcb-rescue:GND-power #PWR0119
-U 1 1 5F58185D
-P 4500 3600
-F 0 "#PWR0119" H 4500 3350 50  0001 C CNN
-F 1 "GND" H 4505 3427 50  0000 C CNN
-F 2 "" H 4500 3600 50  0001 C CNN
-F 3 "" H 4500 3600 50  0001 C CNN
-	1    4500 3600
-	1    0    0    -1
-$EndComp
-Text GLabel 4400 3400 3    50   Input ~ 0
-S0
-Text GLabel 4600 3400 3    50   Input ~ 0
-S1
-$Comp
 L pcb-rescue:D_Small-Device D11
 U 1 1 5F3D080E
@@
 	5150 1800 5150 2250
 Connection ~ 5150 2250
-Wire Wire Line
-	5150 2250 5150 2600
 Wire Wire Line
 	6000 1000 6000 1350
@@
 Text GLabel 1950 2550 3    50   Input ~ 0
 ROW2
-Text GLabel 1750 4800 0    50   Input ~ 0
-S0
 Wire Wire Line
 	1750 5100 1750 5000
@@
 Text GLabel 2200 4150 0    50   Input ~ 0
 reset
-Text GLabel 1750 4900 0    50   Input ~ 0
-S1
 Text GLabel 1750 5800 0    50   Input ~ 0
 COL4
@@
 	6600 2950 5750 2950
 Connection ~ 5750 2950
-Wire Wire Line
-	5750 2950 5200 2950
 $Comp
 L pcb-rescue:VCC-power #PWR0105
 U 1 1 5FE47AAE
-P 1750 3350
-F 0 "#PWR0105" H 1750 3200 50  0001 C CNN
-F 1 "VCC" H 1767 3523 50  0000 C CNN
-F 2 "" H 1750 3350 50  0001 C CNN
-F 3 "" H 1750 3350 50  0001 C CNN
-	1    1750 3350
+P 1850 3300
+F 0 "#PWR0105" H 1850 3150 50  0001 C CNN
+F 1 "VCC" H 1867 3473 50  0000 C CNN
+F 2 "" H 1850 3300 50  0001 C CNN
+F 3 "" H 1850 3300 50  0001 C CNN
+	1    1850 3300
 	1    0    0    -1
 $EndComp
@@
 Text GLabel 3150 5200 2    50   Input ~ 0
 COL5
+Text GLabel 3150 5600 2    50   Input ~ 0
+COL6
+Text GLabel 3150 5500 2    50   Input ~ 0
+COL7
+Text GLabel 3150 5400 2    50   Input ~ 0
+COL8
 Text GLabel 3150 5300 2    50   Input ~ 0
-COL6
-Text GLabel 3150 5400 2    50   Input ~ 0
-COL7
-Text GLabel 3150 5500 2    50   Input ~ 0
-COL8
-Text GLabel 3150 5600 2    50   Input ~ 0
 COL9
 $Comp
-L pcb-rescue:Rotary_Encoder_Switch-Device SW33
-U 1 1 5F50E358
-P 4500 3100
-F 0 "SW33" V 4546 2870 50  0000 R CNN
-F 1 "Rotary_Encoder_Switch" V 4455 2870 50  0000 R CNN
-F 2 "keebio-parts:RotaryEncoder_EC11" H 4350 3260 50  0001 C CNN
-F 3 "~" H 4500 3360 50  0001 C CNN
-	1    4500 3100
-	0    -1   -1   0
-$EndComp
-Wire Wire Line
-	4500 3400 4500 3600
-Wire Wire Line
-	4600 2800 5200 2800
-Wire Wire Line
-	5200 2800 5200 2950
-Connection ~ 5200 2950
-Wire Wire Line
-	5200 2950 5100 2950
-Wire Wire Line
-	4400 2800 4400 2600
-Wire Wire Line
-	4400 2600 5150 2600
-Connection ~ 5150 2600
-Wire Wire Line
-	5150 2600 5150 2650
+L SSD1306-128x64_OLED:SSD1306 Brd1
+U 1 1 5FA7259A
+P 3000 3250
+F 0 "Brd1" V 3046 2972 50  0000 R CNN
+F 1 "SSD1306" V 2955 2972 50  0000 R CNN
+F 2 "SSD1306:128x64OLED" H 3000 3500 50  0001 C CNN
+F 3 "" H 3000 3500 50  0001 C CNN
+	1    3000 3250
+	0    -1   -1   0
+$EndComp
+Wire Wire Line
+	2250 3100 2650 3100
+Text GLabel 2250 3200 0    50   Input ~ 0
+SCL
+Wire Wire Line
+	2650 3200 2250 3200
+Wire Wire Line
+	1850 3400 2650 3400
+$Comp
+L pcb-rescue:GND-power #PWR0115
+U 1 1 5F4567A6
+P 1850 3400
+F 0 "#PWR0115" H 1850 3150 50  0001 C CNN
+F 1 "GND" H 1855 3227 50  0000 C CNN
+F 2 "" H 1850 3400 50  0001 C CNN
+F 3 "" H 1850 3400 50  0001 C CNN
+	1    1850 3400
+	1    0    0    -1
+$EndComp
+Wire Wire Line
+	5150 2250 5150 2650
+Wire Wire Line
+	5100 2950 5750 2950
+NoConn ~ 1750 4800
+NoConn ~ 1750 4900
+NoConn ~ 3150 4800
 $EndSCHEMATC
